File: EB-190/EB-190.kicad_sch (KiCad schematic)
At the start: 144 parts, among them J1 Conn_02x18_Top_Bottom, P1 R_Potentiometer, Q1 NPN, Q2 NPN, Q3 2N4126, SW1 SW_Reed, U1 MC33193

Commit message: EB190  - Finished - Waiting for review
Parts:
- removed L1, L2: L, symbol Device:L
- removed R25: 180R, Resistor_SMD:R_0603_1608Metric, symbol firmlogik-resistor-0603:RES-180R-0603-1P
- removed SW1: SW_Reed, symbol Switch:SW_Reed
- added L5: ~, firmlogik-inductors:Dual Coil with Reed Relay, symbol firmlogik-inductor:DUAL_COIL_AND_REED_RELAY
- renumbered LED2 to LED1, LED1 to LED2, L3 to RLY3
Connections:
- net BLNK_RES: no longer JP1.2 (B)
- net GND: now also Q2.1 (C); no longer Q2.3 (E)
- net RLY_C: no longer RLY3.8
- net at TP47.1: now also L5.2B
- net at TP63.1: now also D1.1 (K); no longer D2.1 (K)
- net at S1.1 (A): now also Q2.3 (E); no longer Q2.1 (C)
- net at F2.1: now also L5.1B, L5.2A, L5.4
- net at TP39.1: now also L5.1A
- net at TP74.1: now also D1.2 (A); no longer D2.2 (A)
- net at TP46.1: now also L5.3
- net at TP62.1: now also D2.2 (A); no longer D1.2 (A)
- net at TP73.1: now also D2.1 (K); no longer D1.1 (K)
Other:
- moved on the sheet: D1, D2, Q2, TP40

Commit message: Fixed a small thing I noticed when the switch was desoldered.
Connections:
- net at Q2.3 (E), S1.1 (A): now also S1.3 (C)
Changed lines of the file:
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@@
   (junction (at 255.778 85.852) (diameter 0) (color 0 0 0 0)
   )
+  (junction (at 85.09 85.598) (diameter 0) (color 0 0 0 0)
+  )
   (junction (at 249.936 49.784) (diameter 0) (color 0 0 0 0)
   )
@@
     (stroke (width 0) (type default))
   )
+  (wire (pts (xy 85.09 80.518) (xy 85.09 85.598))
+    (stroke (width 0) (type default))
+  )
+  (wire (pts (xy 96.52 25.908) (xy 105.156 25.908))
+    (stroke (width 0) (type default))
+  )
+  (wire (pts (xy 250.444 85.852) (xy 255.778 85.852))
+    (stroke (width 0) (type default))
+  )
+  (wire (pts (xy 205.232 104.267) (xy 205.232 105.156))
+    (stroke (width 0) (type default))
+  )
+  (wire (pts (xy 88.392 85.598) (xy 85.09 85.598))
+    (stroke (width 0) (type default))
+  )
+  (wire (pts (xy 249.682 152.4) (xy 252.984 152.4))
+    (stroke (width 0) (type default))
+  )
+  (wire (pts (xy 53.086 52.832) (xy 53.086 50.292))
+    (stroke (width 0) (type default))
+  )
+  (wire (pts (xy 110.744 28.194) (xy 115.062 28.194))
+    (stroke (width 0) (type default))
+  )
+  (wire (pts (xy 226.568 129.286) (xy 226.568 131.826))
+    (stroke (width 0) (type default))
+  )
+  (wire (pts (xy 268.478 49.784) (xy 249.936 49.784))
+    (stroke (width 0) (type default))
+  )
+  (wire (pts (xy 173.99 146.05) (xy 173.99 147.574))
+    (stroke (width 0) (type default))
+  )
+  (wire (pts (xy 203.2 129.286) (xy 203.2 126.492))
+    (stroke (width 0) (type default))
+  )
+  (wire (pts (xy 133.858 85.09) (xy 133.858 67.31))
+    (stroke (width 0) (type default))
+  )
+  (wire (pts (xy 201.676 27.178) (xy 202.946 27.178))
+    (stroke (width 0) (type default))
+  )
+  (wire (pts (xy 202.692 78.74) (xy 202.692 88.9))
+    (stroke (width 0) (type default))
+  )
+  (wire (pts (xy 97.79 122.682) (xy 97.79 107.696))
+    (stroke (width 0) (type default))
+  )
+  (wire (pts (xy 164.084 29.972) (xy 164.084 31.496))
+    (stroke (width 0) (type default))
+  )
+  (wire (pts (xy 231.648 100.33) (xy 231.648 106.172))
+    (stroke (width 0) (type default))
+  )
+  (wire (pts (xy 128.016 47.244) (xy 128.016 49.53))
+    (stroke (width 0) (type default))
+  )
+  (wire (pts (xy 85.09 95.25) (xy 109.22 95.25))
+    (stroke (width 0) (type default))
+  )
+  (wire (pts (xy 227.838 32.258) (xy 227.838 34.29))
+    (stroke (width 0) (type default))
+  )
+  (wire (pts (xy 18.542 40.132) (xy 23.114 40.132))
+    (stroke (width 0) (type default))
+  )
+  (wire (pts (xy 117.602 25.908) (xy 117.602 28.194))
+    (stroke (width 0) (type default))
+  )
+  (wire (pts (xy 215.392 129.286) (xy 215.392 130.048))
+    (stroke (width 0) (type default))
+  )
+  (wire (pts (xy 110.744 33.274) (xy 110.744 42.672))
+    (stroke (width 0) (type default))
+  )
+  (wire (pts (xy 264.922 39.878) (xy 266.192 39.878))
+    (stroke (width 0) (type default))
+  )
+  (wire (pts (xy 104.902 75.438) (xy 104.902 83.058))
+    (stroke (width 0) (type default))
+  )
+  (wire (pts (xy 122.682 27.94) (xy 122.682 28.194))
+    (stroke (width 0) (type default))
+  )
+  (wire (pts (xy 16.51 22.352) (xy 30.734 22.352))
+    (stroke (width 0) (type default))
+  )
+  (wire (pts (xy 128.016 57.15) (xy 128.016 63.5))
+    (stroke (width 0) (type default))
+  )
   (wire (pts (xy 85.09 85.598) (xy 85.09 95.25))
     (stroke (width 0) (type default))
   )
-  (wire (pts (xy 96.52 25.908) (xy 105.156 25.908))
-    (stroke (width 0) (type default))
-  )
-  (wire (pts (xy 250.444 85.852) (xy 255.778 85.852))
-    (stroke (width 0) (type default))
-  )
-  (wire (pts (xy 205.232 104.267) (xy 205.232 105.156))
-    (stroke (width 0) (type default))
-  )
-  (wire (pts (xy 88.392 85.598) (xy 85.09 85.598))
-    (stroke (width 0) (type default))
-  )
-  (wire (pts (xy 249.682 152.4) (xy 252.984 152.4))
-    (stroke (width 0) (type default))
-  )
-  (wire (pts (xy 53.086 52.832) (xy 53.086 50.292))
-    (stroke (width 0) (type default))
-  )
-  (wire (pts (xy 110.744 28.194) (xy 115.062 28.194))
-    (stroke (width 0) (type default))
-  )
-  (wire (pts (xy 226.568 129.286) (xy 226.568 131.826))
-    (stroke (width 0) (type default))
-  )
-  (wire (pts (xy 268.478 49.784) (xy 249.936 49.784))
-    (stroke (width 0) (type default))
-  )
-  (wire (pts (xy 173.99 146.05) (xy 173.99 147.574))
-    (stroke (width 0) (type default))
-  )
-  (wire (pts (xy 203.2 129.286) (xy 203.2 126.492))
-    (stroke (width 0) (type default))
-  )
-  (wire (pts (xy 133.858 85.09) (xy 133.858 67.31))
-    (stroke (width 0) (type default))
-  )
-  (wire (pts (xy 201.676 27.178) (xy 202.946 27.178))
-    (stroke (width 0) (type default))
-  )
-  (wire (pts (xy 202.692 78.74) (xy 202.692 88.9))
-    (stroke (width 0) (type default))
-  )
-  (wire (pts (xy 97.79 122.682) (xy 97.79 107.696))
-    (stroke (width 0) (type default))
-  )
-  (wire (pts (xy 164.084 29.972) (xy 164.084 31.496))
-    (stroke (width 0) (type default))
-  )
-  (wire (pts (xy 231.648 100.33) (xy 231.648 106.172))
-    (stroke (width 0) (type default))
-  )
-  (wire (pts (xy 128.016 47.244) (xy 128.016 49.53))
-    (stroke (width 0) (type default))
-  )
-  (wire (pts (xy 85.09 95.25) (xy 109.22 95.25))
-    (stroke (width 0) (type default))
-  )
-  (wire (pts (xy 227.838 32.258) (xy 227.838 34.29))
-    (stroke (width 0) (type default))
-  )
-  (wire (pts (xy 18.542 40.132) (xy 23.114 40.132))
-    (stroke (width 0) (type default))
-  )
-  (wire (pts (xy 117.602 25.908) (xy 117.602 28.194))
-    (stroke (width 0) (type default))
-  )
-  (wire (pts (xy 215.392 129.286) (xy 215.392 130.048))
-    (stroke (width 0) (type default))
-  )
-  (wire (pts (xy 110.744 33.274) (xy 110.744 42.672))
-    (stroke (width 0) (type default))
-  )
-  (wire (pts (xy 264.922 39.878) (xy 266.192 39.878))
-    (stroke (width 0) (type default))
-  )
-  (wire (pts (xy 104.902 75.438) (xy 104.902 83.058))
-    (stroke (width 0) (type default))
-  )
-  (wire (pts (xy 122.682 27.94) (xy 122.682 28.194))
-    (stroke (width 0) (type default))
-  )
-  (wire (pts (xy 16.51 22.352) (xy 30.734 22.352))
-    (stroke (width 0) (type default))
-  )
-  (wire (pts (xy 128.016 57.15) (xy 128.016 63.5))
-    (stroke (width 0) (type default))
-  )
   (wire (pts (xy 212.852 126.492) (xy 215.392 126.492))
     (stroke (width 0) (type default))
@@
     (stroke (width 0) (type default))
   )
+  (wire (pts (xy 85.09 80.518) (xy 88.392 80.518))
+    (stroke (width 0) (type default))
+  )
