File: EB-190/EB-190.kicad_pcb (KiCad board)
At the start: 2 copper layers, 234 x 199.8 mm, 141 parts, among them J1 Conn_02x18_Top_Bottom, P1 R_Potentiometer, Q1 NPN, Q2 NPN, Q3 2N4126, U1 MC33193

Commit message: EB190  - Finished - Waiting for review
Parts:
- removed R25: 180R, Resistor_SMD:R_0603_1608Metric
- added G***: LOGO, LOGO, F.Cu at (294.0, 57.7)
- added L5: ~, firmlogik-inductors:Dual Coil with Reed Relay, F.Cu at (189.4, 104.0)
- added kibuzzard-65B90473: G***, kibuzzard-65B90473, F.Cu at (302.5, 41.9)
- moved D1 38.3 mm to (133.5, 220.7), turned to 180 degrees
- moved D2 38.2 mm to (171.4, 220.7), turned to 0 degrees
- moved TP45 17.9 mm to (189.1, 117.5)
- moved R9 17.0 mm to (284.5, 181.6)
- moved TP39 9.79 mm to (171.1, 141.2)
- moved TP46 9.79 mm to (189.1, 141.2)
- moved TP47 9.79 mm to (207.1, 141.2)
- moved D8 8.12 mm to (230.5, 58.5)
- moved R1 6.60 mm to (113.3, 121.7)
- moved D5 6.22 mm to (305.6, 179.8)
- moved TP35 5.46 mm to (238.3, 172.7)
- moved R8 5.33 mm to (303.9, 80.1)
- moved TP40 4.34 mm to (228.9, 188.7)
- moved F2 2.99 mm to (175.5, 117.5), turned to 0 degrees
- moved LED2 2.97 mm to (139.3, 122.2), turned to 0 degrees
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- renumbered L3 to RLY3
Connections:
- LED1 pad 1: /BLNK_LED_A -> Net-(LED1-K)
- LED1 pad 2: Net-(LED1-A) -> /BLNK_LED_A
- LED2 pad 1: Net-(LED1-A) -> /BLNK_LED_A
- LED2 pad 2: /BLNK_LED_A -> Net-(LED1-K)
- Q2 pad 1: Net-(Q2-C) -> GND
- Q2 pad 3: GND -> Net-(Q2-E)
- S1 pad 1: Net-(Q2-C) -> Net-(Q2-E)
- S1 pad 4: Net-(LED1-A) -> Net-(LED1-K)
- TP62 pad 1: Net-(D1-A) -> Net-(D2-A)
- TP63 pad 1: Net-(D2-K) -> Net-(D1-K)
- TP73 pad 1: Net-(D1-K) -> Net-(D2-K)
- TP74 pad 1: Net-(D2-A) -> Net-(D1-A)
- TP8 pad 1: Net-(LED1-A) -> Net-(LED1-K)
Routing:
- net Net-(LED1-K): track 0.00 -> 91.7 mm
- net Net-(LED1-A): track 91.1 -> 0.00 mm
- net Net-(F2-Pad1): track 0.00 -> 61.6 mm
- net Net-(L5-Pad3): track 0.00 -> 53.9 mm
- net Net-(L5-Pad1A): track 0.00 -> 45.1 mm
- net /I4: track 229.4 -> 189.7 mm
- net Net-(L5-Pad2B): track 0.00 -> 38.4 mm
- net Net-(Q2-E): track 0.00 -> 19.2 mm
- net Net-(Q2-C): track 19.2 -> 0.00 mm
- net Net-(I5--): track 28.4 -> 11.4 mm
- net GND: track 696.4 -> 685.4 mm
- net Net-(D8-A): track 21.0 -> 11.6 mm
- net Net-(R7-Pad1): track 32.2 -> 41.1 mm
- net Net-(F2-Pad2): track 0.00 -> 8.64 mm
- net Net-(L4-+): track 49.7 -> 58.3 mm
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Other:
- board text added: "+12V"
- board text added: "+PS 1"
- board text added: "1000μF"
- board text added: "100R"
- board text added: "14V 80mA"
- board text added: "1K"
- board text added: "270R"
- board text added: "680"
- board text added: "BUZZER"
- board text added: "C"
- board text added: "CURRENT SENSE"
- board text added: "D4"
- board text added: "D5"
- board text added: "FLASHER"
- board text added: "HEATER"
- board text added: "I OUT"
- board text added: "I1"
- board text added: "I2"
- board text added: "I3"
- board text added: "I4"
- board text added: "L"
- board text added: "L1"
- board text added: "L2"
- board text added: "L3"
- board text added: "L4"
- board text added: "LED"
- board text added: "NC NO"
- board text added: "NEON"
- board text added: "OFF"
- board text added: "P1"
- board text added: "PUSH BUTTON SWITCHES"
- board text added: "Q1"
- board text added: "R"
- board text added: "R1"
- board text added: "R5"
- board text added: "R6 10R"
- board text added: "R7 500R"
- board text added: "R8 1K"
- board text added: "REED SWITCH"
- board text added: "RELAY SPDT"
- board text added: "S1"
- board text added: "S2"
- board text added: "S3"
- board text added: "S4"
- board text added: "S5"
- board text added: "S6"
- board text added: "SOLENOID"
- board text added: "THERMAL SWITCH"
- board text added: "THERMISTOR"
- board text added: "TOGGLE SWITCHES"

Commit message: Fixed a small thing I noticed when the switch was desoldered.
Connections:
- S1 pad 3: unconnected-(S1-C-Pad3) -> Net-(Q2-E)
Routing:
- net Net-(Q2-E): track 19.2 -> 30.6 mm

Commit message: Updated some mistakes
Other:
- board text added: "V1.0 2024"
Changed lines of the file:
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@@
     (effects (font (size 2 2) (thickness 0.5) bold) (justify left bottom))
+  )
+  (gr_text "V1.0 2024" (at 287.782 36.83) (layer "F.SilkS")
+    (effects (font (size 1.5 1.5) (thickness 0.3) bold) (justify left bottom))
   )
   (gr_text "1000μF" (at 164.338 203.581) (layer "F.SilkS")
